File: ardentis/MCU-Storage-PWR.kicad_sch (KiCad schematic)
At the start: 38 parts, among them IC3 RT6150B-33GQW, J1 USB_MicroB_Receptical_5pin, J2 Micro_SD_Card, J4 Conn_01x02_Pin, U1 ESP32-S3-MINI-1, Y1 32.768kHz(NC)

Commit message: Initial code
Initial code. Theoretically will work but not tested due to lack of hardware and updates to PCB.
Parts:
- removed J4: Conn_01x02_Pin, symbol Connector:Conn_01x02_Pin
- removed JP4, JP5: SolderJumper_3_Bridged12, symbol Jumper:SolderJumper_3_Bridged12
- removed R1, R2: 0(NC), symbol Device:R_Small
- removed R3: NC, symbol Device:R_Small
- removed Y1: 32.768kHz(NC), symbol Device:Crystal_Small
- added J1: Conn_01x02_Pin, Library:TestPoint_2Pads_Pitch2.54mm_Drill0.8mm, symbol Library:Conn_01x02_Pin
- added J4: Screw_Terminal_01x04, Library:TB00150004BE, symbol Library:Screw_Terminal_01x04
- added JP3: Jumper_2_Small_Open, Library:SolderJumper-2_P1.3mm_Open_TrianglePad1.0x1.5mm, symbol Library:Jumper_2_Small_Open
- added JP4: SolderJumper_3_Open, Library:SolderJumper-3_P2.0mm_Open_TrianglePad1.0x1.5mm, symbol Library:SolderJumper_3_Open
- C11: renamed from C13; footprint (none) -> Library:C_0805_2012Metric_Pad1.18x1.45mm_HandSolder; symbol Device:C_Small -> Library:C_Small; Manufacturer_Name Murata Electronics -> Samsung Electro-Mechanics; Manufacturer_Part_Number GRM21BZ70J226ME44L -> CL21X226MQQNNNE; Price 0.293 -> 0.2; SPN (none) -> 1276-3031-2-ND
- C12: footprint (none) -> Library:C_0805_2012Metric_Pad1.18x1.45mm_HandSolder; symbol Device:C_Small -> Library:C_Small; Manufacturer_Name Murata Electronics -> Samsung Electro-Mechanics; Manufacturer_Part_Number GRM21BZ70J226ME44L -> CL21X226MQQNNNE; Price 0.293 -> 0.2; SPN (none) -> 1276-3031-2-ND
- C13: renamed from C4; footprint (none) -> Library:C_0805_2012Metric_Pad1.18x1.45mm_HandSolder; symbol Device:C_Small -> Library:C_Small; Manufacturer_Name Murata Electronics -> Samsung Electro-Mechanics; Manufacturer_Part_Number GRM21BZ70J226ME44L -> CL21X226MQQNNNE; Price 0.293 -> 0.2; SPN (none) -> 1276-3031-2-ND; Var (none) -> Variant Ground(-!) Flight(+!)
- C14: renamed from C5; footprint (none) -> Library:C_0805_2012Metric_Pad1.18x1.45mm_HandSolder; symbol Device:C_Small -> Library:C_Small; Manufacturer_Part_Number 08053C104KAT2A -> KGM21NR71H104KT; Price 0.07 -> 0.12; SPN (none) -> 478-KGM21NR71H104KTTR-ND; Var (none) -> Variant Ground(-!) Flight(+!)
- C15: renamed from C3; footprint (none) -> Library:C_0805_2012Metric_Pad1.18x1.45mm_HandSolder; symbol Device:C_Small -> Library:C_Small; Manufacturer_Part_Number 08053C104KAT2A -> KGM21NR71H104KT; Price 0.07 -> 0.12; SPN (none) -> 478-KGM21NR71H104KTTR-ND
- C16: renamed from C1; footprint (none) -> Library:C_0805_2012Metric_Pad1.18x1.45mm_HandSolder; symbol Device:C_Small -> Library:C_Small; Manufacturer_Part_Number 08053C104KAT2A -> KGM21NR71H104KT; Price 0.07 -> 0.12; SPN (none) -> 478-KGM21NR71H104KTTR-ND
- C17: renamed from C2; footprint (none) -> Library:C_0805_2012Metric_Pad1.18x1.45mm_HandSolder; symbol Device:C_Small -> Library:C_Small; Manufacturer_Name Murata Electronics -> Samsung Electro-Mechanics; Manufacturer_Part_Number GRM21BZ70J226ME44L -> CL21X226MQQNNNE; Price 0.293 -> 0.2; SPN (none) -> 1276-3031-2-ND
- J5: renamed from J2; footprint (none) -> Library:MEM20670218000A; symbol Connector:Micro_SD_Card -> Library:Micro_SD_Card; Price 1.62 -> 1.60; SPN (none) -> 2073-MEM2067-02-180-00-ATR-ND; Var (none) -> Variant Ground(-!) Flight(+!)
- J6: renamed from J1; footprint (none) -> Library:UJ2MIBHGSMTTR; symbol Connector:USB_B_Micro -> Library:USB_B_Micro; Price 0.58 -> 0.67; SPN (none) -> 2223-UJ2-MIBH-G-SMT-TR-ND
- JP1: renamed from JP2; value RESET -> RST; footprint TestPoint:TestPoint_2Pads_Pitch2.54mm_Drill0.8mm -> Library:TestPoint_2Pads_Pitch2.54mm_Drill0.8mm; symbol Jumper:Jumper_2_Small_Open -> Library:Jumper_2_Small_Open
- JP2: renamed from JP1; footprint TestPoint:TestPoint_2Pads_Pitch2.54mm_Drill0.8mm -> Library:TestPoint_2Pads_Pitch2.54mm_Drill0.8mm; symbol Jumper:Jumper_2_Small_Open -> Library:Jumper_2_Small_Open
- JP5: renamed from JP9; footprint (none) -> Library:SolderJumper-3_P2.0mm_Open_TrianglePad1.0x1.5mm; symbol Jumper:SolderJumper_3_Bridged12 -> Library:SolderJumper_3_Bridged12
- JP6: renamed from JP10; footprint (none) -> Library:SolderJumper-3_P2.0mm_Open_TrianglePad1.0x1.5mm; symbol Jumper:SolderJumper_3_Bridged12 -> Library:SolderJumper_3_Bridged12
- L1: renamed from L2; footprint (none) -> Inductor_SMD:L_1008_2520Metric_Pad1.43x2.20mm_HandSolder; symbol Device:L_Small -> Library:L_Small; Manufacturer_Name Bourns -> INPAQ Technology Co., Ltd; Manufacturer_Part_Number SRN2510F-2R2M -> WIP252012S-2R2MLDG; Price 0.168 -> 0.15; SPN (none) -> 3526-WIP252012S-2R2MLDGTR-ND
- R10: renamed from R17; footprint (none) -> Library:R_0805_2012Metric_Pad1.20x1.40mm_HandSolder; symbol Device:R_Small -> Library:R_Small; Manufacturer_Name KOA Speer -> YAGEO; Manufacturer_Part_Number RK73B2ATTD103J -> RC0805JR-0710KL; Price 0.024 -> 0.019; SPN (none) -> 311-10KARTR-ND
- R11: renamed from R5; footprint (none) -> Library:R_0805_2012Metric_Pad1.20x1.40mm_HandSolder; symbol Device:R_Small -> Library:R_Small; Manufacturer_Name KOA Speer -> Panasonic Electronic Components; Manufacturer_Part_Number RK73Z2ATTD -> ERJ-6GEY0R00V; Price 0.024 -> 0.16; SPN (none) -> P0.0ATR-ND
- R12: renamed from R7; footprint (none) -> Library:R_0805_2012Metric_Pad1.20x1.40mm_HandSolder; symbol Device:R_Small -> Library:R_Small; Manufacturer_Name KOA Speer -> YAGEO; Manufacturer_Part_Number RK73B2ATTD103J -> RC0805JR-0710KL; Price 0.024 -> 0.019; SPN (none) -> 311-10KARTR-ND; Var (none) -> Variant Ground(-!) Flight(+!)
- R13: renamed from R4; footprint (none) -> Library:R_0805_2012Metric_Pad1.20x1.40mm_HandSolder; symbol Device:R_Small -> Library:R_Small; Manufacturer_Name KOA Speer -> Panasonic Electronic Components; Manufacturer_Part_Number RK73Z2ATTD -> ERJ-6GEY0R00V; Price 0.024 -> 0.16; SPN (none) -> P0.0ATR-ND
- R14: renamed from R8; footprint (none) -> Library:R_0805_2012Metric_Pad1.20x1.40mm_HandSolder; symbol Device:R_Small -> Library:R_Small; Manufacturer_Name KOA Speer -> YAGEO; Manufacturer_Part_Number RK73B2ATTD103J -> RC0805JR-0710KL; Price 0.024 -> 0.019; SPN (none) -> 311-10KARTR-ND; Var (none) -> Variant Ground(-!) Flight(+!)
- R15: renamed from R6; footprint (none) -> Library:R_0805_2012Metric_Pad1.20x1.40mm_HandSolder; symbol Device:R_Small -> Library:R_Small; Manufacturer_Name KOA Speer -> YAGEO; Manufacturer_Part_Number RK73B2ATTD103J -> RC0805JR-0710KL; Price 0.024 -> 0.019; SPN (none) -> 311-10KARTR-ND
- R16: renamed from R9; footprint (none) -> Library:R_0805_2012Metric_Pad1.20x1.40mm_HandSolder; symbol Device:R_Small -> Library:R_Small; Manufacturer_Name KOA Speer -> YAGEO; Manufacturer_Part_Number RK73B2ATTD103J -> RC0805JR-0710KL; Price 0.024 -> 0.019; SPN (none) -> 311-10KARTR-ND; Var (none) -> Variant Ground(-!) Flight(+!)
- R17: renamed from R10; footprint (none) -> Library:R_0805_2012Metric_Pad1.20x1.40mm_HandSolder; symbol Device:R_Small -> Library:R_Small; Manufacturer_Name KOA Speer -> YAGEO; Manufacturer_Part_Number RK73B2ATTD103J -> RC0805JR-0710KL; Price 0.024 -> 0.019; SPN (none) -> 311-10KARTR-ND; Var (none) -> Variant Ground(-!) Flight(+!)
- R18: renamed from R11; footprint (none) -> Library:R_0805_2012Metric_Pad1.20x1.40mm_HandSolder; symbol Device:R_Small -> Library:R_Small; Manufacturer_Name KOA Speer -> YAGEO; Manufacturer_Part_Number RK73B2ATTD103J -> RC0805JR-0710KL; Price 0.024 -> 0.019; SPN (none) -> 311-10KARTR-ND; Var (none) -> Variant Ground(-!) Flight(+!)
- R19: renamed from R12; footprint (none) -> Library:R_0805_2012Metric_Pad1.20x1.40mm_HandSolder; symbol Device:R_Small -> Library:R_Small; Manufacturer_Name KOA Speer -> YAGEO; Manufacturer_Part_Number RK73B2ATTD103J -> RC0805JR-0710KL; Price 0.024 -> 0.019; SPN (none) -> 311-10KARTR-ND; Var (none) -> Variant Ground(-!) Flight(+!)
- R3: renamed from R13; footprint (none) -> Library:R_0805_2012Metric_Pad1.20x1.40mm_HandSolder; symbol Device:R_Small -> Library:R_Small; Manufacturer_Name KOA Speer -> YAGEO; Manufacturer_Part_Number RK73B2ATTD103J -> RC0805JR-0710KL; Price 0.024 -> 0.019; SPN (none) -> 311-10KARTR-ND; Var (none) -> Variant Ground(-!) Flight(+!)
- R6: renamed from R16; footprint (none) -> Library:R_0805_2012Metric_Pad1.20x1.40mm_HandSolder; symbol Device:R_Small -> Library:R_Small; Manufacturer_Name KOA Speer -> YAGEO; Manufacturer_Part_Number RK73B2ATTD103J -> RC0805JR-0710KL; Price 0.024 -> 0.019; SPN (none) -> 311-10KARTR-ND
- R7: renamed from R15; footprint (none) -> Library:R_0805_2012Metric_Pad1.20x1.40mm_HandSolder; symbol Device:R_Small -> Library:R_Small; Manufacturer_Name KOA Speer -> YAGEO; Manufacturer_Part_Number RK73B2ATTD103J -> RC0805JR-0710KL; Price 0.024 -> 0.019; SPN (none) -> 311-10KARTR-ND
- R8: renamed from R14; footprint (none) -> Library:R_0805_2012Metric_Pad1.20x1.40mm_HandSolder; symbol Device:R_Small -> Library:R_Small; Manufacturer_Name KOA Speer -> YAGEO; Manufacturer_Part_Number RK73B2ATTD103J -> RC0805JR-0710KL; Price 0.024 -> 0.019; SPN (none) -> 311-10KARTR-ND; Var (none) -> Variant Ground(-!) Flight(+!)
- R9: renamed from R18; footprint (none) -> Library:R_0805_2012Metric_Pad1.20x1.40mm_HandSolder; symbol Device:R_Small -> Library:R_Small; Manufacturer_Name KOA Speer -> YAGEO; Manufacturer_Part_Number RK73B2ATTD103J -> RC0805JR-0710KL; Price 0.024 -> 0.019; SPN (none) -> 311-10KARTR-ND
- U7: renamed from IC3; footprint SON50P250X250X80-11N-D -> Library:SON50P250X250X80-11N-D; symbol RT6150B-33GQW:RT6150B-33GQW -> Library:RT6150B-33GQW; Price 4.35 -> 4.62; SPN (none) -> RT6150B-33GQWTR-ND
- U8: renamed from U1; value ESP32-S3-MINI-1 -> ESP32-S3-MINI-1-N8; footprint RF_Module:ESP32-S2-MINI-1 -> Library:ESP32-S3-MINI-1; symbol RF_Module:ESP32-S3-MINI-1 -> Library:ESP32-S3-MINI-1; Manufacturer_Part_Number ESP32-MINI-1-N4 -> 1965-ESP32-S3-MINI-1-N4R2TR-ND; Price 3.51 -> 8.4
Connections:
- net +3V3: no longer J5.1 (DAT2), J5.2 (DAT3/CD), J5.3 (CMD), R12.2, R14.2, R16.2, U8.28 (IO33), U8.29 (IO34), U8.31 (IO35)
- net +5V: now also JP4.3 (B)
- net +BATT: now also J4.2 (Pin_2), J4.3 (Pin_3), JP3.1 (A); no longer C12.1, R7.2, U7.5 (VIN), U7.6 (EN), U7.8 (VINA)
- net ADC0: now also U8.18 (IO14); no longer U8.5 (IO1)
- net EN: now also C15.1, JP1.2 (B), R15.1
- net GND: now also U7.7 (PS), J4.4 (Pin_4)
- net SD.D1: no longer U8.34 (IO38)
- net IO15: now reaches U8.19 (IO15)
- net USB_MCU.D+: now reaches R11.1, U8.24 (USB_D+)
- net IO6: now reaches U8.10 (IO6)
- net IO7: now reaches U8.11 (IO7)
- net IO11: now reaches U8.15 (IO11)
- net IO12: now reaches U8.16 (IO12)
- net IO13: now reaches U8.17 (IO13)
- net IO16: now reaches U8.20 (IO16)
- net TX1: now reaches JP6.2 (C), U8.21 (IO17)
- net RX1: now reaches JP5.2 (C), U8.22 (IO18)
- net USB_MCU.D-: now reaches R13.1, U8.23 (USB_D-)
- net IO21: now reaches U8.25 (IO21)
- net IO47: now reaches U8.27 (IO47)
- net IO48: now reaches U8.30 (IO48)
- net IO39: now reaches U8.35 (IO39)
- net IO40: now reaches U8.36 (IO40)
- net IO41: now reaches U8.37 (IO41)
- net IO42: now reaches U8.38 (IO42)
- net TX0: now reaches U8.39 (TXD0)
- net TX0: now also J1.2 (Pin_2)
- net BOOT: now reaches JP2.2 (B), U8.4 (IO0)
- net RX0: now reaches U8.40 (RXD0)
- net RX0: now also J1.1 (Pin_1)
- net IO4: now reaches U8.8 (IO4)
- net IO5: now reaches U8.9 (IO5)
- new net +VSW: J4.1 (Pin_1), JP3.2 (B), JP4.1 (A), R7.2
- new net IO1: U8.5 (IO1)
- new net IO33: U8.28 (IO33)
- new net IO38: U8.34 (IO38)
- new net SD.CMD: J5.3 (CMD), R16.2, U8.31 (IO35)
- new net SD.D2: J5.1 (DAT2), R12.2
- new net SD.D3: J5.2 (DAT3/CD), R14.2, U8.29 (IO34)
- new net VCC: C12.1, JP4.2 (C), U7.5 (VIN), U7.6 (EN), U7.8 (VINA)
- no-connect marks 1 -> 4
Other:
- company: (none) -> CU INSPACE
- moved on the sheet: C13, C14, J5, R11, R12, R13, R14, R16, R17, R18, R19, R3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
